File: pcb_ruler.kicad_pcb (KiCad board)
At the start: 2 copper layers, 160 x 38 mm, 13 parts

Commit message: v2.0
Other:
- board text added: "ZIG PCB Ruler v.2.0 M. Lundberg 2024"
- board text removed: "ZIG PCB Ruler v.1.0 M. Lundberg 2023"
